File: ft2232h_esp32.sch (KiCad schematic (older format))
At the start: 72 parts, among them J1 USB_C_Receptacle_USB2.0, Q1 S8050, Q2 S8050, SW1 SW_SPDT, U1 ESP32FullConnector, U10 USBLC6-2SC6-Power_Protection, U11 USBLC6-2SC6-Power_Protection, U12 USBLC6-2SC6-Power_Protection, U13 USBLC6-2SC6-Power_Protection, U2 ESP32FullConnector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

Commit message: V0
Parts:
- removed R1: 0, Resistor_SMD:R_0603_1608Metric, symbol Device:R
- removed R10, R8, R9: 33R(1%), Resistor_SMD:R_0603_1608Metric, symbol Device:R
- removed R2, R5, R7: 10k(1%), Resistor_SMD:R_0603_1608Metric, symbol Device:R
- removed R6: 2.2k(1%), Resistor_SMD:R_0603_1608Metric, symbol Device:R
- removed U4: 93C56-C173182, Package_SO:SOP-8_3.76x4.96mm_P1.27mm, symbol Memory_EEPROM:93CxxC
Changed lines of the file:
@@
-$EndComp
-$Comp
-L Memory_EEPROM:93CxxC U4
-U 1 1 6063278B
-P 4170 7160
-F 0 "U4" H 3560 7000 50  0000 C CNN
-F 1 "93C56-C173182" H 3740 6880 50  0000 C CNN
-F 2 "Package_SO:SOP-8_3.76x4.96mm_P1.27mm" H 4170 7160 50  0001 C CNN
-F 3 "http://ww1.microchip.com/downloads/en/DeviceDoc/20001749K.pdf" H 4170 7160 50  0001 C CNN
-	1    4170 7160
-	1    0    0    -1
 $EndComp
 $Comp
@@
 	0    -1   -1   0
 $EndComp
-$Comp
-L Device:R R1
-U 1 1 6061510A
-P 870 3730
-F 0 "R1" V 870 3740 50  0000 C CNN
-F 1 "0" V 754 3730 50  0000 C CNN
-F 2 "Resistor_SMD:R_0603_1608Metric" V 800 3730 50  0001 C CNN
-F 3 "~" H 870 3730 50  0001 C CNN
-F 4 "C21189" H 870 3730 50  0001 C CNN "LCSC"
-	1    870  3730
-	0    1    1    0
-$EndComp
-Connection ~ 1020 3730
 $Comp
 L Connector:USB_C_Receptacle_USB2.0 J1
@@
 	1    3400 3580
 	0    -1   -1   0
-$EndComp
-$Comp
-L Device:R R8
-U 1 1 606271FF
-P 3290 4680
-F 0 "R8" V 3290 4690 50  0000 C CNN
-F 1 "33R(1%)" V 3240 4950 50  0000 C CNN
-F 2 "Resistor_SMD:R_0603_1608Metric" V 3220 4680 50  0001 C CNN
-F 3 "~" H 3290 4680 50  0001 C CNN
-F 4 "C23140" H 3290 4680 50  0001 C CNN "LCSC"
-	1    3290 4680
-	0    1    1    0
-$EndComp
-Wire Wire Line
-	3440 4680 3700 4680
-Text GLabel 3140 4680 0    50   Input ~ 0
-EECS
-$Comp
-L Device:R R9
-U 1 1 6062990B
-P 3290 4780
-F 0 "R9" V 3290 4790 50  0000 C CNN
-F 1 "33R(1%)" V 3240 5050 50  0000 C CNN
-F 2 "Resistor_SMD:R_0603_1608Metric" V 3220 4780 50  0001 C CNN
-F 3 "~" H 3290 4780 50  0001 C CNN
-F 4 "C23140" H 3290 4780 50  0001 C CNN "LCSC"
-	1    3290 4780
-	0    1    1    0
-$EndComp
-$Comp
-L Device:R R10
-U 1 1 6062A110
-P 3290 4880
-F 0 "R10" V 3290 4890 50  0000 C CNN
-F 1 "33R(1%)" V 3240 5150 50  0000 C CNN
-F 2 "Resistor_SMD:R_0603_1608Metric" V 3220 4880 50  0001 C CNN
-F 3 "~" H 3290 4880 50  0001 C CNN
-F 4 "C23140" H 3290 4880 50  0001 C CNN "LCSC"
-	1    3290 4880
-	0    1    1    0
-$EndComp
-Wire Wire Line
-	3440 4780 3700 4780
-Wire Wire Line
-	3440 4880 3700 4880
-Text GLabel 3140 4780 0    50   Input ~ 0
-EECLK
-Text GLabel 3140 4880 0    50   Input ~ 0
-EEDATA
-Text GLabel 4650 7060 2    50   Input ~ 0
-EECLK
-$Comp
-L Device:R R5
-U 1 1 6063D805
-P 4570 6910
-F 0 "R5" V 4570 6870 50  0000 L CNN
-F 1 "10k(1%)" V 4470 6870 50  0000 L CNN
-F 2 "Resistor_SMD:R_0603_1608Metric" V 4500 6910 50  0001 C CNN
-F 3 "~" H 4570 6910 50  0001 C CNN
-F 4 "C25804" H 4570 6910 50  0001 C CNN "LCSC"
-	1    4570 6910
-	1    0    0    -1
-$EndComp
-Wire Wire Line
-	4570 7060 4650 7060
-Connection ~ 4570 7060
-$Comp
-L power:+3V3 #PWR0114
-U 1 1 6064AEC4
-P 4570 6760
-F 0 "#PWR0114" H 4570 6610 50  0001 C CNN
-F 1 "+3V3" H 4585 6933 50  0000 C CNN
-F 2 "" H 4570 6760 50  0001 C CNN
-F 3 "" H 4570 6760 50  0001 C CNN
-	1    4570 6760
-	1    0    0    -1
-$EndComp
-$Comp
-L Device:R R6
-U 1 1 6064C7A0
-P 4720 7260
-F 0 "R6" V 4720 7260 50  0000 C CNN
-F 1 "2.2k(1%)" V 4820 7260 50  0000 C CNN
-F 2 "Resistor_SMD:R_0603_1608Metric" V 4650 7260 50  0001 C CNN
-F 3 "~" H 4720 7260 50  0001 C CNN
-F 4 "C4190" H 4720 7260 50  0001 C CNN "LCSC"
-	1    4720 7260
-	0    1    1    0
-$EndComp
-Text GLabel 5060 7160 2    50   Input ~ 0
-EEDATA
-Wire Wire Line
-	4870 7260 4870 7160
-Wire Wire Line
-	4570 7160 4870 7160
-Connection ~ 4870 7160
-Wire Wire Line
-	4870 7160 5000 7160
-$Comp
-L Device:R R7
-U 1 1 6064FF94
-P 5000 7010
-F 0 "R7" V 5000 6970 50  0000 L CNN
-F 1 "10k(1%)" V 5090 6910 50  0000 L CNN
-F 2 "Resistor_SMD:R_0603_1608Metric" V 4930 7010 50  0001 C CNN
-F 3 "~" H 5000 7010 50  0001 C CNN
-F 4 "C25804" H 5000 7010 50  0001 C CNN "LCSC"
-	1    5000 7010
-	1    0    0    -1
-$EndComp
-Connection ~ 5000 7160
-Wire Wire Line
-	5000 7160 5060 7160
-Wire Wire Line
-	4570 6760 5000 6760
-Wire Wire Line
-	5000 6760 5000 6860
-Connection ~ 4570 6760
-Wire Wire Line
-	3530 6980 3530 7060
-$Comp
-L Device:R R2
-U 1 1 60635E67
-P 3530 6830
-F 0 "R2" V 3530 6790 50  0000 L CNN
-F 1 "10k(1%)" V 3430 6700 50  0000 L CNN
-F 2 "Resistor_SMD:R_0603_1608Metric" V 3460 6830 50  0001 C CNN
-F 3 "~" H 3530 6830 50  0001 C CNN
-F 4 "C25804" H 3530 6830 50  0001 C CNN "LCSC"
-	1    3530 6830
-	1    0    0    -1
-$EndComp
-$Comp
-L power:+3V3 #PWR0115
-U 1 1 60632D75
-P 3530 6680
-F 0 "#PWR0115" H 3530 6530 50  0001 C CNN
-F 1 "+3V3" H 3545 6853 50  0000 C CNN
-F 2 "" H 3530 6680 50  0001 C CNN
-F 3 "" H 3530 6680 50  0001 C CNN
-	1    3530 6680
-	1    0    0    -1
-$EndComp
-Text GLabel 3530 7060 0    50   Input ~ 0
-EECS
-Wire Wire Line
-	3770 7060 3530 7060
-$Comp
-L power:+3V3 #PWR0116
-U 1 1 6065B4A8
-P 3770 7160
-F 0 "#PWR0116" H 3770 7010 50  0001 C CNN
-F 1 "+3V3" H 3785 7333 50  0000 C CNN
-F 2 "" H 3770 7160 50  0001 C CNN
-F 3 "" H 3770 7160 50  0001 C CNN
-	1    3770 7160
-	-1   0    0    1
-$EndComp
-$Comp
-L power:GND #PWR0117
-U 1 1 6065CA7B
-P 4170 7460
-F 0 "#PWR0117" H 4170 7210 50  0001 C CNN
-F 1 "GND" H 4175 7287 50  0000 C CNN
-F 2 "" H 4170 7460 50  0001 C CNN
-F 3 "" H 4170 7460 50  0001 C CNN
-	1    4170 7460
-	1    0    0    -1
 $EndComp
 $Comp
@@
 Text GLabel 1220 1810 2    50   Input ~ 0
 ESPTX
-$Comp
-L power:+3V3 #PWR0152
-U 1 1 60732C49
-P 4170 6860
-F 0 "#PWR0152" H 4170 6710 50  0001 C CNN
-F 1 "+3V3" H 4185 7033 50  0000 C CNN
-F 2 "" H 4170 6860 50  0001 C CNN
-F 3 "" H 4170 6860 50  0001 C CNN
-	1    4170 6860
-	1    0    0    -1
-$EndComp
 Text GLabel 8950 4570 1    50   Input ~ 0
 ESPRX
