File: ft2232h_esp32.sch (KiCad schematic (older format))
At the start: 68 parts, among them J1 USB_C_Receptacle_USB2.0, Q1 S8050, Q2 S8050, SW1 SW_SPDT, U1 ESP32FullConnector, U2 ESP32FullConnector, U3 USBLC6-2SC6-Power_Protection, U4 93C56-C173182, U5 FT2232HL, U6 ESP32FullConnector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

Commit message: update
Parts:
- removed D1: ESDLC5V0PB8, Package_DFN_QFN:UDFN-9_1.0x3.8mm_P0.5mm, symbol Power_Protection:ESDLC5V0PB8
- added H5, H6, H7, H8: MountingHole, MountingHole:MountingHole_2.2mm_M2, symbol Mechanical:MountingHole
- added U10, U11, U12, U13: USBLC6-2SC6-Power_Protection, Package_TO_SOT_SMD:SOT-23-6, symbol KisonCommon:USBLC6-2SC6-Power_Protection
- R19, R20: footprint (none) -> Resistor_SMD:R_0603_1608Metric
Connections:
- wire segments 68 -> 69
Other:
- moved on the sheet: C17, C18, C19, C20, C21, C22, D5, L1, R18, R19, R20, R21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

Commit message: layout
Parts:
- L1: footprint Inductor_SMD:L_01005_0402Metric -> Inductor_SMD:L_1008_2520Metric
- U10, U11, U12, U13, U3: footprint Package_TO_SOT_SMD:SOT-23-6 -> KisonCommon:USBLC6-2P6-SOT666
Connections:
- net +3V3: no longer U10.5 (VBUS), U11.5 (VBUS), U12.5 (VBUS), U13.5 (VBUS)
- net GND: now also C21.1, U3.2 (GND)
- net EN renamed nTRST
Changed lines of the file:
@@
 IO0
 Text GLabel 6020 620  2    50   Input ~ 0
-EN
-Text GLabel 6920 610  2    50   Input ~ 0
 nTRST
-Text GLabel 6920 610  0    50   Input ~ 0
-EN
 Text GLabel 1220 800  2    50   Input ~ 0
 nTRST
@@
 F 0 "L1" V 10200 2030 50  0000 C CNN
 F 1 "2.2uh" V 10270 2030 50  0000 C CNN
-F 2 "Inductor_SMD:L_01005_0402Metric" H 10320 2030 50  0001 C CNN
+F 2 "Inductor_SMD:L_1008_2520Metric" H 10320 2030 50  0001 C CNN
 F 3 "~" H 10320 2030 50  0001 C CNN
 	1    10320 2030
@@
 F 0 "U3" H 1370 5251 50  0000 C CNN
 F 1 "USBLC6-2SC6-Power_Protection" H 1370 5160 50  0000 C CNN
-F 2 "Package_TO_SOT_SMD:SOT-23-6" H 620 4970 50  0001 C CNN
+F 2 "KisonCommon:USBLC6-2P6-SOT666" H 620 4970 50  0001 C CNN
 F 3 "" H 1570 4920 50  0001 C CNN
 	1    1370 4570
@@
 F 0 "U11" H 8480 3911 50  0000 C CNN
 F 1 "USBLC6-2SC6-Power_Protection" H 8480 3840 50  0000 C CNN
-F 2 "Package_TO_SOT_SMD:SOT-23-6" H 7730 3630 50  0001 C CNN
+F 2 "KisonCommon:USBLC6-2P6-SOT666" H 7730 3630 50  0001 C CNN
 F 3 "" H 8680 3580 50  0001 C CNN
 	1    8480 3230
@@
 TXD
 $Comp
-L power:+3V3 #PWR013
-U 1 1 6074579A
-P 8480 2730
-F 0 "#PWR013" H 8480 2580 50  0001 C CNN
-F 1 "+3V3" H 8495 2903 50  0000 C CNN
-F 2 "" H 8480 2730 50  0001 C CNN
-F 3 "" H 8480 2730 50  0001 C CNN
-	1    8480 2730
-	0    1    1    0
-$EndComp
-$Comp
 L power:GND #PWR015
 U 1 1 60753364
@@
 F 0 "U12" H 9890 4291 50  0000 C CNN
 F 1 "USBLC6-2SC6-Power_Protection" H 9890 4220 50  0000 C CNN
-F 2 "Package_TO_SOT_SMD:SOT-23-6" H 9140 4010 50  0001 C CNN
+F 2 "KisonCommon:USBLC6-2P6-SOT666" H 9140 4010 50  0001 C CNN
 F 3 "" H 10090 3960 50  0001 C CNN
 	1    9890 3610
 	1    0    0    -1
-$EndComp
-$Comp
-L power:+3V3 #PWR014
-U 1 1 60753370
-P 9890 3110
-F 0 "#PWR014" H 9890 2960 50  0001 C CNN
-F 1 "+3V3" H 9905 3283 50  0000 C CNN
-F 2 "" H 9890 3110 50  0001 C CNN
-F 3 "" H 9890 3110 50  0001 C CNN
-	1    9890 3110
-	0    1    1    0
 $EndComp
 $Comp
@@
 F 0 "U10" H 8450 5351 50  0000 C CNN
 F 1 "USBLC6-2SC6-Power_Protection" H 8450 5280 50  0000 C CNN
-F 2 "Package_TO_SOT_SMD:SOT-23-6" H 7700 5070 50  0001 C CNN
+F 2 "KisonCommon:USBLC6-2P6-SOT666" H 7700 5070 50  0001 C CNN
 F 3 "" H 8650 5020 50  0001 C CNN
 	1    8450 4670
 	1    0    0    -1
-$EndComp
-$Comp
-L power:+3V3 #PWR011
-U 1 1 607A234E
-P 8450 4170
-F 0 "#PWR011" H 8450 4020 50  0001 C CNN
-F 1 "+3V3" H 8465 4343 50  0000 C CNN
-F 2 "" H 8450 4170 50  0001 C CNN
-F 3 "" H 8450 4170 50  0001 C CNN
-	1    8450 4170
-	0    1    1    0
 $EndComp
 $Comp
@@
 F 0 "U13" H 9890 5771 50  0000 C CNN
 F 1 "USBLC6-2SC6-Power_Protection" H 9890 5700 50  0000 C CNN
-F 2 "Package_TO_SOT_SMD:SOT-23-6" H 9140 5490 50  0001 C CNN
+F 2 "KisonCommon:USBLC6-2P6-SOT666" H 9140 5490 50  0001 C CNN
 F 3 "" H 10090 5440 50  0001 C CNN
 	1    9890 5090
 	1    0    0    -1
-$EndComp
-$Comp
-L power:+3V3 #PWR016
-U 1 1 607A4C5B
-P 9890 4590
-F 0 "#PWR016" H 9890 4440 50  0001 C CNN
-F 1 "+3V3" H 9905 4763 50  0000 C CNN
-F 2 "" H 9890 4590 50  0001 C CNN
-F 3 "" H 9890 4590 50  0001 C CNN
-	1    9890 4590
-	0    1    1    0
 $EndComp
 Text GLabel 10390 3710 3    50   Input ~ 0
@@
 Text GLabel 9390 5190 3    50   Input ~ 0
 IO0
+$Comp
+L power:GND #PWR0150
+U 1 1 6087C1CA
+P 6550 7180
+F 0 "#PWR0150" H 6550 6930 50  0001 C CNN
+F 1 "GND" H 6555 7007 50  0000 C CNN
+F 2 "" H 6550 7180 50  0001 C CNN
+F 3 "" H 6550 7180 50  0001 C CNN
+	1    6550 7180
+	1    0    0    -1
+$EndComp
+$Comp
+L power:GND #PWR0151
+U 1 1 608B5D46
+P 1370 5070
+F 0 "#PWR0151" H 1370 4820 50  0001 C CNN
+F 1 "GND" V 1375 4942 50  0000 R CNN
+F 2 "" H 1370 5070 50  0001 C CNN
+F 3 "" H 1370 5070 50  0001 C CNN
+	1    1370 5070
+	1    0    0    -1
+$EndComp
 $EndSCHEMATC

Commit message: Fix Crystal
Parts:
- added R22, R23, R24: 0, Resistor_SMD:R_0603_1608Metric, symbol Device:R
- C18, C20: value 22pf -> 22uf
- U1, U6, U7: footprint KisonCommon:jtag1.27-12 -> KisonCommon:jtag1.27-10
- U2: footprint Connector_Molex:Molex_CLIK-Mate_502382-1270_1x12-1MP_P1.25mm_Vertical -> Connector_Molex:Molex_CLIK-Mate_502382-1070_1x10-1MP_P1.25mm_Vertical
- X1: footprint Oscillator:Oscillator_SMD_Abracon_ASCO-4Pin_1.6x1.2mm -> Oscillator:Oscillator_SMD_Fordahl_DFAS15-4Pin_5.0x3.2mm
Connections:
- net +3V3: now also U4.8 (VCC)
- net 3v3OUT: now also U1.7 (3V3), U2.7 (3V3)
- net GND: now also R24.2; no longer R20.2
- net IO0: now also U1.8 (IO0), U2.8 (IO0)
- net TCK: now also U1.4 (TCLK), U2.4 (TCLK)
- net TDI: now also U1.3 (TDI), U2.3 (TDI)
- net TDO: now also U1.6 (TDO), U2.6 (TDO)
- net TMS: now also U1.5 (TMS), U2.5 (TMS)
- net ESPRX: now reaches U1.10 (RX)
- net ESPRX: now also U10.3 (IO2), U10.4 (IO2), U2.10 (RX), R22.1
- net ESPTX: now reaches U1.9 (TX)
- net ESPTX: now also U10.1 (IO1), U10.6 (IO1), U2.9 (TX), R23.1
- net at C19.2, R19.1, U9.5 (FB): now also R20.2; no longer R20.1
- removed net RXD: U10.3 (IO2), U10.4 (IO2), U5.39 (BDBUS1)
- removed net TXD: U10.1 (IO1), U10.6 (IO1), U5.38 (BDBUS0)
- new net: R20.1, R24.1
- new net 2232RX: R23.2, U5.39 (BDBUS1)
- new net 2232TX: R22.2, U5.38 (BDBUS0)
Other:
- moved on the sheet: R20
Changed lines of the file:
@@
 F 0 "U1" H 1010 1434 50  0000 C CNN
 F 1 "ESP32FullConnector" H 1010 1343 50  0000 C CNN
-F 2 "KisonCommon:jtag1.27-12" H 1200 1010 50  0001 C CNN
+F 2 "KisonCommon:jtag1.27-10" H 1200 1010 50  0001 C CNN
 F 3 "" H 1200 1010 50  0001 C CNN
 	1    1200 1010
-	1    0    0    -1
-$EndComp
-$Comp
-L KisonCommon:ESP32FullConnector U2
-U 1 1 60623F40
-P 1200 1660
-F 0 "U2" H 1010 2084 50  0000 C CNN
-F 1 "ESP32FullConnector" H 1010 1993 50  0000 C CNN
-F 2 "Connector_Molex:Molex_CLIK-Mate_502382-1270_1x12-1MP_P1.25mm_Vertical" H 1200 1660 50  0001 C CNN
-F 3 "" H 1200 1660 50  0001 C CNN
-	1    1200 1660
-	1    0    0    -1
-$EndComp
-$Comp
-L Interface_USB:FT2232HL U5
-U 1 1 60625869
-P 4900 3980
-F 0 "U5" H 4900 6361 50  0000 C CNN
-F 1 "FT2232HL" H 4900 6270 50  0000 C CNN
-F 2 "Package_QFP:LQFP-64_10x10mm_P0.5mm" H 4900 3980 50  0001 C CNN
-F 3 "https://www.ftdichip.com/Support/Documents/DataSheets/ICs/DS_FT2232H.pdf" H 4900 3980 50  0001 C CNN
-	1    4900 3980
 	1    0    0    -1
 $EndComp
@@
 U 1 1 6063278B
 P 4170 7160
-F 0 "U4" H 4000 7580 50  0000 C CNN
-F 1 "93C56-C173182" H 4030 7510 50  0000 C CNN
+F 0 "U4" H 3560 7000 50  0000 C CNN
+F 1 "93C56-C173182" H 3740 6880 50  0000 C CNN
 F 2 "Package_SO:SOP-8_3.76x4.96mm_P1.27mm" H 4170 7160 50  0001 C CNN
 F 3 "http://ww1.microchip.com/downloads/en/DeviceDoc/20001749K.pdf" H 4170 7160 50  0001 C CNN
@@
 Connection ~ 5200 6180
 Connection ~ 4500 6180
-Wire Wire Line
-	4500 6180 4300 6180
-Connection ~ 4600 6180
-Wire Wire Line
-	4600 6180 4500 6180
 Connection ~ 4700 6180
-Wire Wire Line
-	4700 6180 4600 6180
 Connection ~ 4800 6180
 Wire Wire Line
@@
 Wire Wire Line
 	4900 6180 4800 6180
-Connection ~ 5000 6180
-Wire Wire Line
-	5000 6180 4900 6180
 Connection ~ 5100 6180
 Wire Wire Line
-	5100 6180 5000 6180
-Wire Wire Line
-	3700 5780 3700 6180
-Wire Wire Line
 	3700 6180 4300 6180
-Connection ~ 4300 6180
 $Comp
 L power:+1V8 #PWR0119
@@
 	5100 1780 5200 1780
 Connection ~ 5200 1780
-Wire Wire Line
-	5200 1780 5300 1780
-Connection ~ 5300 1780
-Wire Wire Line
-	5300 1780 5400 1780
 $Comp
 L power:+3V3 #PWR0120
@@
 	1    0    0    -1
 $EndComp
-Connection ~ 5400 1780
 Text GLabel 6100 2080 2    50   Input ~ 0
 TCK
@@
 Text GLabel 6100 2580 2    50   Input ~ 0
 nTRST
-Text GLabel 6100 3880 2    50   Input ~ 0
-TXD
-Text GLabel 6100 3980 2    50   Input ~ 0
-RXD
 $Comp
 L Transistor_BJT:S8050 Q1
@@
 Text GLabel 1220 1450 2    50   Input ~ 0
 nTRST
-Text GLabel 800  1800 0    50   Input ~ 0
+Text GLabel 800  1720 0    50   Input ~ 0
 IO0
-Text GLabel 800  1150 0    50   Input ~ 0
+Text GLabel 800  1070 0    50   Input ~ 0
 IO0
-Text GLabel 1220 1080 2    50   Input ~ 0
-TXD
-Text GLabel 1220 1730 2    50   Input ~ 0
-TXD
-Text GLabel 800  1080 0    50   Input ~ 0
-RXD
-Text GLabel 800  1730 0    50   Input ~ 0
-RXD
-Text GLabel 800  870  0    50   Input ~ 0
+Text GLabel 800  890  0    50   Input ~ 0
 TCK
-Text GLabel 800  1520 0    50   Input ~ 0
+Text GLabel 800  1540 0    50   Input ~ 0
 TCK
-Text GLabel 800  940  0    50   Input ~ 0
+Text GLabel 800  980  0    50   Input ~ 0
 TDO
-Text GLabel 800  1590 0    50   Input ~ 0
+Text GLabel 800  1630 0    50   Input ~ 0
 TDO
 $Comp
@@
 	0    1    1    0
 $EndComp
-Text GLabel 1220 870  2    50   Input ~ 0
+Text GLabel 1220 890  2    50   Input ~ 0
 TDI
-Text GLabel 1220 1520 2    50   Input ~ 0
+Text GLabel 1220 1540 2    50   Input ~ 0
 TDI
-Text GLabel 1220 940  2    50   Input ~ 0
+Text GLabel 1220 980  2    50   Input ~ 0
 TMS
-Text GLabel 1220 1590 2    50   Input ~ 0
+Text GLabel 1220 1630 2    50   Input ~ 0
 TMS
 Text GLabel 6100 4280 2    50   Input ~ 0
@@
 F 0 "U6" H 1230 7264 50  0000 C CNN
 F 1 "ESP32FullConnector" H 1230 7173 50  0000 C CNN
-F 2 "KisonCommon:jtag1.27-12" H 1420 6840 50  0001 C CNN
+F 2 "KisonCommon:jtag1.27-10" H 1420 6840 50  0001 C CNN
 F 3 "" H 1420 6840 50  0001 C CNN
 	1    1420 6840
@@
 F 0 "U7" H 1240 7934 50  0000 C CNN
 F 1 "ESP32FullConnector" H 1240 7843 50  0000 C CNN
-F 2 "KisonCommon:jtag1.27-12" H 1430 7510 50  0001 C CNN
+F 2 "KisonCommon:jtag1.27-10" H 1430 7510 50  0001 C CNN
 F 3 "" H 1430 7510 50  0001 C CNN
 	1    1430 7510
@@
 F 0 "X1" H 3364 5406 50  0000 L CNN
 F 1 "ASCO" H 3364 5315 50  0000 L CNN
-F 2 "Oscillator:Oscillator_SMD_Abracon_ASCO-4Pin_1.6x1.2mm" H 3020 5010 50  0001 C CNN
+F 2 "Oscillator:Oscillator_SMD_Fordahl_DFAS15-4Pin_5.0x3.2mm" H 3020 5010 50  0001 C CNN
 F 3 "https://abracon.com/Oscillators/ASCO.pdf" H 2695 5485 50  0001 C CNN
 	1    2920 5360
@@
 	0    -1   -1   0
 $EndComp
-Text GLabel 1220 1010 2    50   Input ~ 0
+Text GLabel 1220 1070 2    50   Input ~ 0
 3v3OUT
 $Comp
@@
 Connection ~ 10470 2030
 $Comp
-L Device:R R20
-U 1 1 60848352
-P 10470 2560
-F 0 "R20" V 10470 2510 50  0000 L CNN
-F 1 "22k" V 10390 2520 50  0000 L CNN
-F 2 "Resistor_SMD:R_0603_1608Metric" V 10400 2560 50  0001 C CNN
-F 3 "~" H 10470 2560 50  0001 C CNN
-	1    10470 2560
-	-1   0    0    -1
-$EndComp
-$Comp
 L power:GND #PWR08
 U 1 1 60848F79
-P 10470 2710
-F 0 "#PWR08" H 10470 2460 50  0001 C CNN
-F 1 "GND" H 10475 2537 50  0000 C CNN
-F 2 "" H 10470 2710 50  0001 C CNN
-F 3 "" H 10470 2710 50  0001 C CNN
-	1    10470 2710
+P 10770 2710
+F 0 "#PWR08" H 10770 2460 50  0001 C CNN
+F 1 "GND" H 10775 2537 50  0000 C CNN
+F 2 "" H 10770 2710 50  0001 C CNN
+F 3 "" H 10770 2710 50  0001 C CNN
+	1    10770 2710
 	-1   0    0    -1
 $EndComp
@@
 P 10770 1880
 F 0 "C18" H 10600 1960 50  0000 L CNN
-F 1 "22pf" H 10580 1780 50  0000 L CNN
+F 1 "22uf" H 10580 1780 50  0000 L CNN
 F 2 "Capacitor_SMD:C_0603_1608Metric" H 10808 1730 50  0001 C CNN
 F 3 "~" H 10770 1880 50  0001 C CNN
@@
 P 10470 1880
 F 0 "C20" H 10310 1960 50  0000 L CNN
-F 1 "22pf" H 10280 1780 50  0000 L CNN
+F 1 "22uf" H 10280 1780 50  0000 L CNN
 F 2 "Capacitor_SMD:C_0603_1608Metric" H 10508 1730 50  0001 C CNN
 F 3 "~" H 10470 1880 50  0001 C CNN
@@
 Wire Wire Line
 	10300 2330 10470 2330
-Text GLabel 1220 1660 2    50   Input ~ 0
+Text GLabel 1220 1720 2    50   Input ~ 0
 3v3OUT
 Text GLabel 8980 3130 1    50   Input ~ 0
@@
 Text GLabel 9390 3510 1    50   Input ~ 0
 TCK
-Text GLabel 8950 4570 1    50   Input ~ 0
-RXD
 Text GLabel 9390 4990 1    50   Input ~ 0
 IO0
-Text GLabel 7950 4570 1    50   Input ~ 0
-TXD
 $Comp
 L power:GND #PWR015
@@
 Text GLabel 10390 5190 3    50   Input ~ 0
 TDO
-Text GLabel 8950 4770 3    50   Input ~ 0
-RXD
-Text GLabel 7950 4770 3    50   Input ~ 0
-TXD
 Text GLabel 10390 4990 1    50   Input ~ 0
 TDO
@@
 	1    0    0    -1
 $EndComp
+Text GLabel 6100 3880 2    50   Input ~ 0
+2232TX
+Text GLabel 6950 3450 0    50   Input ~ 0
+2232TX
+$Comp
+L Device:R R22
+U 1 1 607147ED
+P 7100 3450
+F 0 "R22" V 7100 3450 50  0000 C CNN
+F 1 "0" V 6984 3450 50  0000 C CNN
+F 2 "Resistor_SMD:R_0603_1608Metric" V 7030 3450 50  0001 C CNN
+F 3 "~" H 7100 3450 50  0001 C CNN
+	1    7100 3450
+	0    1    1    0
+$EndComp
+Text GLabel 7250 3450 2    50   Input ~ 0
+ESPRX
+$Comp
+L Device:R R23
+U 1 1 6071BB77
+P 7100 3570
+F 0 "R23" V 7100 3570 50  0000 C CNN
+F 1 "0" V 6984 3570 50  0000 C CNN
+F 2 "Resistor_SMD:R_0603_1608Metric" V 7030 3570 50  0001 C CNN
+F 3 "~" H 7100 3570 50  0001 C CNN
+	1    7100 3570
+	0    1    -1   0
+$EndComp
+Text GLabel 6100 3980 2    50   Input ~ 0
+2232RX
+Text GLabel 6950 3570 0    50   Input ~ 0
+2232RX
+Text GLabel 7250 3570 2    50   Input ~ 0
+ESPTX
+Text GLabel 1220 1160 2    50   Input ~ 0
+ESPTX
+Text GLabel 800  1160 0    50   Input ~ 0
+ESPRX
+Text GLabel 800  1810 0    50   Input ~ 0
+ESPRX
+Text GLabel 1220 1810 2    50   Input ~ 0
+ESPTX
+$Comp
+L power:+3V3 #PWR0152
+U 1 1 60732C49
+P 4170 6860
+F 0 "#PWR0152" H 4170 6710 50  0001 C CNN
+F 1 "+3V3" H 4185 7033 50  0000 C CNN
+F 2 "" H 4170 6860 50  0001 C CNN
+F 3 "" H 4170 6860 50  0001 C CNN
+	1    4170 6860
+	1    0    0    -1
+$EndComp
+Text GLabel 8950 4570 1    50   Input ~ 0
+ESPRX
+Text GLabel 7950 4570 1    50   Input ~ 0
+ESPTX
+Text GLabel 7950 4770 3    50   Input ~ 0
+ESPTX
+Text GLabel 8950 4770 3    50   Input ~ 0
+ESPRX
+Connection ~ 5400 1780
+Connection ~ 5300 1780
+Wire Wire Line
+	5300 1780 5400 1780
+Wire Wire Line
+	5200 1780 5300 1780
+Connection ~ 4300 6180
+Wire Wire Line
+	5100 6180 5000 6180
+Wire Wire Line
+	5000 6180 4900 6180
+Connection ~ 5000 6180
+Wire Wire Line
+	4700 6180 4600 6180
+Wire Wire Line
+	4600 6180 4500 6180
+Connection ~ 4600 6180
+Wire Wire Line
+	3700 5780 3700 6180
+Wire Wire Line
+	4500 6180 4300 6180
+$Comp
+L Interface_USB:FT2232HL U5
+U 1 1 60625869
+P 4900 3980
+F 0 "U5" H 4900 6361 50  0000 C CNN
+F 1 "FT2232HL" H 4900 6270 50  0000 C CNN
+F 2 "Package_QFP:LQFP-64_10x10mm_P0.5mm" H 4900 3980 50  0001 C CNN
+F 3 "https://www.ftdichip.com/Support/Documents/DataSheets/ICs/DS_FT2232H.pdf" H 4900 3980 50  0001 C CNN
+	1    4900 3980
+	1    0    0    -1
+$EndComp
+$Comp
+L KisonCommon:ESP32FullConnector U2
+U 1 1 60623F40
+P 1200 1660
+F 0 "U2" H 1010 2084 50  0000 C CNN
+F 1 "ESP32FullConnector" H 1010 1993 50  0000 C CNN
+F 2 "Connector_Molex:Molex_CLIK-Mate_502382-1070_1x10-1MP_P1.25mm_Vertical" H 1200 1660 50  0001 C CNN
+F 3 "" H 1200 1660 50  0001 C CNN
+	1    1200 1660
+	1    0    0    -1
+$EndComp
+$Comp
+L Device:R R20
+U 1 1 60848352
+P 10620 2410
+F 0 "R20" V 10620 2360 50  0000 L CNN
+F 1 "22k" V 10540 2370 50  0000 L CNN
+F 2 "Resistor_SMD:R_0603_1608Metric" V 10550 2410 50  0001 C CNN
+F 3 "~" H 10620 2410 50  0001 C CNN
+	1    10620 2410
+	0    1    -1   0
+$EndComp
+$Comp
+L Device:R R24
+U 1 1 60722D2E
+P 10770 2560
+F 0 "R24" V 10770 2490 50  0000 L CNN
+F 1 "0" H 10840 2515 50  0000 L CNN
+F 2 "Resistor_SMD:R_0603_1608Metric" V 10700 2560 50  0001 C CNN
+F 3 "~" H 10770 2560 50  0001 C CNN
+	1    10770 2560
+	1    0    0    -1
+$EndComp
