File: ft2232h_esp32.sch (KiCad schematic (older format))
At the start: 78 parts, among them J1 USB_C_Receptacle_USB2.0, Q1 S8050, Q2 S8050, SW1 SW_SPDT, U1 ESP32FullConnector, U10 USBLC6-2SC6-Power_Protection, U11 USBLC6-2SC6-Power_Protection, U12 USBLC6-2SC6-Power_Protection, U13 USBLC6-2SC6-Power_Protection, U2 ESP32FullConnector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

Commit message: Add LCSC
Parts:
- C1, C2, C3, C4: LCSC (none) -> C19666
- C10, C11, C12, C13, C14, C15, C5, C6, C9: LCSC (none) -> C14663
- C17, C21: LCSC (none) -> C15849
- C18, C20, C22: LCSC (none) -> C59461
- C19: LCSC (none) -> C1653
- C7, C8: LCSC (none) -> C1648
- D2: LCSC (none) -> C72043
- D3: LCSC (none) -> C72041
- D4: LCSC (none) -> C2286
- D5: LCSC (none) -> C72038
- Q1, Q2: LCSC (none) -> C2150
- R1, R22, R23, R24: LCSC (none) -> C21189
- R10, R8, R9: LCSC (none) -> C23140
- R11: LCSC (none) -> C22790
- R12, R18: LCSC (none) -> C21190
- R13, R14, R19: LCSC (none) -> C25803
- R15, R2, R21, R5, R7: LCSC (none) -> C25804
- R16, R17, R6: LCSC (none) -> C4190
- R20: LCSC (none) -> C31850
- R3, R4: LCSC (none) -> C23186
Changed lines of the file:
@@
 F 2 "Capacitor_SMD:C_0603_1608Metric" H 3348 1140 50  0001 C CNN
 F 3 "~" H 3310 1290 50  0001 C CNN
+F 4 "C19666" H 3310 1290 50  0001 C CNN "LCSC"
 	1    3310 1290
 	1    0    0    -1
@@
 F 2 "Capacitor_SMD:C_0603_1608Metric" H 3918 1140 50  0001 C CNN
 F 3 "~" H 3880 1290 50  0001 C CNN
+F 4 "C14663" H 3880 1290 50  0001 C CNN "LCSC"
 	1    3880 1290
 	1    0    0    -1
@@
 F 2 "Capacitor_SMD:C_0603_1608Metric" H 3648 1220 50  0001 C CNN
 F 3 "~" H 3610 1370 50  0001 C CNN
+F 4 "C14663" H 3610 1370 50  0001 C CNN "LCSC"
 	1    3610 1370
 	1    0    0    -1
@@
 F 2 "Capacitor_SMD:C_0603_1608Metric" H 3058 1210 50  0001 C CNN
 F 3 "~" H 3020 1360 50  0001 C CNN
+F 4 "C19666" H 3020 1360 50  0001 C CNN "LCSC"
 	1    3020 1360
 	1    0    0    -1
@@
 F 2 "Capacitor_SMD:C_0603_1608Metric" H 3138 1930 50  0001 C CNN
 F 3 "~" H 3100 2080 50  0001 C CNN
+F 4 "C19666" H 3100 2080 50  0001 C CNN "LCSC"
 	1    3100 2080
 	0    1    1    0
@@
 F 2 "Capacitor_SMD:C_0603_1608Metric" H 3138 2130 50  0001 C CNN
 F 3 "~" H 3100 2280 50  0001 C CNN
+F 4 "C19666" H 3100 2280 50  0001 C CNN "LCSC"
 	1    3100 2280
 	0    1    1    0
@@
 F 2 "Resistor_SMD:R_0603_1608Metric" V 800 3730 50  0001 C CNN
 F 3 "~" H 870 3730 50  0001 C CNN
+F 4 "C21189" H 870 3730 50  0001 C CNN "LCSC"
 	1    870  3730
 	0    1    1    0
@@
 F 2 "Resistor_SMD:R_0603_1608Metric" V 1700 2430 50  0001 C CNN
 F 3 "~" H 1770 2430 50  0001 C CNN
+F 4 "C23186" H 1770 2430 50  0001 C CNN "LCSC"
 	1    1770 2430
 	0    1    1    0
@@
 F 2 "Resistor_SMD:R_0603_1608Metric" V 1700 2530 50  0001 C CNN
 F 3 "~" H 1770 2530 50  0001 C CNN
+F 4 "C23186" H 1770 2530 50  0001 C CNN "LCSC"
 	1    1770 2530
 	0    1    -1   0
@@
 F 2 "Resistor_SMD:R_0603_1608Metric" V 3480 3380 50  0001 C CNN
 F 3 "~" H 3550 3380 50  0001 C CNN
+F 4 "C22790" H 3550 3380 50  0001 C CNN "LCSC"
 	1    3550 3380
 	0    1    1    0
@@
 F 2 "Resistor_SMD:R_0603_1608Metric" V 3480 3580 50  0001 C CNN
 F 3 "~" H 3550 3580 50  0001 C CNN
+F 4 "C21190" H 3550 3580 50  0001 C CNN "LCSC"
 	1    3550 3580
 	0    1    -1   0
@@
 F 2 "Resistor_SMD:R_0603_1608Metric" V 3220 4680 50  0001 C CNN
 F 3 "~" H 3290 4680 50  0001 C CNN
+F 4 "C23140" H 3290 4680 50  0001 C CNN "LCSC"
 	1    3290 4680
 	0    1    1    0
@@
 F 2 "Resistor_SMD:R_0603_1608Metric" V 3220 4780 50  0001 C CNN
 F 3 "~" H 3290 4780 50  0001 C CNN
+F 4 "C23140" H 3290 4780 50  0001 C CNN "LCSC"
 	1    3290 4780
 	0    1    1    0
@@
 F 2 "Resistor_SMD:R_0603_1608Metric" V 3220 4880 50  0001 C CNN
 F 3 "~" H 3290 4880 50  0001 C CNN
+F 4 "C23140" H 3290 4880 50  0001 C CNN "LCSC"
 	1    3290 4880
 	0    1    1    0
@@
 F 2 "Resistor_SMD:R_0603_1608Metric" V 4500 6910 50  0001 C CNN
 F 3 "~" H 4570 6910 50  0001 C CNN
+F 4 "C25804" H 4570 6910 50  0001 C CNN "LCSC"
 	1    4570 6910
 	1    0    0    -1
@@
 F 2 "Resistor_SMD:R_0603_1608Metric" V 4650 7260 50  0001 C CNN
 F 3 "~" H 4720 7260 50  0001 C CNN
+F 4 "C4190" H 4720 7260 50  0001 C CNN "LCSC"
 	1    4720 7260
 	0    1    1    0
@@
 F 2 "Resistor_SMD:R_0603_1608Metric" V 4930 7010 50  0001 C CNN
 F 3 "~" H 5000 7010 50  0001 C CNN
+F 4 "C25804" H 5000 7010 50  0001 C CNN "LCSC"
 	1    5000 7010
 	1    0    0    -1
@@
 F 2 "Resistor_SMD:R_0603_1608Metric" V 3460 6830 50  0001 C CNN
 F 3 "~" H 3530 6830 50  0001 C CNN
+F 4 "C25804" H 3530 6830 50  0001 C CNN "LCSC"
 	1    3530 6830
 	1    0    0    -1
@@
 F 2 "Package_TO_SOT_SMD:SOT-23" H 6120 745 50  0001 L CIN
 F 3 "http://www.unisonic.com.tw/datasheet/S8050.pdf" H 5920 820 50  0001 L CNN
+F 4 "C2150" H 5920 820 50  0001 C CNN "LCSC"
 	1    5920 820
 	1    0    0    -1
@@
 F 2 "Package_TO_SOT_SMD:SOT-23" H 6120 1265 50  0001 L CIN
 F 3 "http://www.unisonic.com.tw/datasheet/S8050.pdf" H 5920 1340 50  0001 L CNN
+F 4 "C2150" H 5920 1340 50  0001 C CNN "LCSC"
 	1    5920 1340
 	1    0    0    1
@@
 F 2 "Resistor_SMD:R_0603_1608Metric" V 5500 820 50  0001 C CNN
 F 3 "~" H 5570 820 50  0001 C CNN
+F 4 "C25803" H 5570 820 50  0001 C CNN "LCSC"
 	1    5570 820
 	0    1    1    0
@@
 F 2 "Resistor_SMD:R_0603_1608Metric" V 5500 1340 50  0001 C CNN
 F 3 "~" H 5570 1340 50  0001 C CNN
+F 4 "C25803" H 5570 1340 50  0001 C CNN "LCSC"
 	1    5570 1340
 	0    1    1    0
@@
 F 2 "Capacitor_SMD:C_0603_1608Metric" H 2408 5210 50  0001 C CNN
 F 3 "~" H 2370 5360 50  0001 C CNN
+F 4 "C1648" H 2370 5360 50  0001 C CNN "LCSC"
 	1    2370 5360
 	0    1    1    0
@@
 F 2 "Capacitor_SMD:C_0603_1608Metric" H 3358 5360 50  0001 C CNN
 F 3 "~" H 3320 5510 50  0001 C CNN
+F 4 "C1648" H 3320 5510 50  0001 C CNN "LCSC"
 	1    3320 5510
 	1    0    0    -1
@@
 F 2 "Capacitor_SMD:C_0603_1608Metric" H 7798 1710 50  0001 C CNN
 F 3 "~" H 7760 1860 50  0001 C CNN
+F 4 "C14663" H 7760 1860 50  0001 C CNN "LCSC"
 	1    7760 1860
 	1    0    0    -1
@@
 F 2 "Capacitor_SMD:C_0603_1608Metric" H 8108 1710 50  0001 C CNN
 F 3 "~" H 8070 1860 50  0001 C CNN
+F 4 "C14663" H 8070 1860 50  0001 C CNN "LCSC"
 	1    8070 1860
 	1    0    0    -1
@@
 F 2 "Capacitor_SMD:C_0603_1608Metric" H 8378 1710 50  0001 C CNN
 F 3 "~" H 8340 1860 50  0001 C CNN
+F 4 "C14663" H 8340 1860 50  0001 C CNN "LCSC"
 	1    8340 1860
 	1    0    0    -1
@@
 F 2 "Capacitor_SMD:C_0603_1608Metric" H 8658 1710 50  0001 C CNN
 F 3 "~" H 8620 1860 50  0001 C CNN
+F 4 "C14663" H 8620 1860 50  0001 C CNN "LCSC"
 	1    8620 1860
 	1    0    0    -1
@@
 F 2 "Capacitor_SMD:C_0603_1608Metric" H 7538 1710 50  0001 C CNN
 F 3 "~" H 7500 1860 50  0001 C CNN
+F 4 "C14663" H 7500 1860 50  0001 C CNN "LCSC"
 	1    7500 1860
 	1    0    0    -1
@@
 F 2 "Capacitor_SMD:C_0603_1608Metric" H 7278 1710 50  0001 C CNN
 F 3 "~" H 7240 1860 50  0001 C CNN
+F 4 "C14663" H 7240 1860 50  0001 C CNN "LCSC"
 	1    7240 1860
 	1    0    0    -1
@@
 F 2 "Capacitor_SMD:C_0603_1608Metric" H 7018 1710 50  0001 C CNN
 F 3 "~" H 6980 1860 50  0001 C CNN
+F 4 "C14663" H 6980 1860 50  0001 C CNN "LCSC"
 	1    6980 1860
 	1    0    0    -1
@@
 F 2 "LED_SMD:LED_0603_1608Metric" H 6710 5180 50  0001 C CNN
 F 3 "~" H 6710 5180 50  0001 C CNN
+F 4 "C2286" H 6710 5180 50  0001 C CNN "LCSC"
 	1    6710 5180
 	1    0    0    -1
@@
 F 2 "LED_SMD:LED_0603_1608Metric" H 6700 4990 50  0001 C CNN
 F 3 "~" H 6700 4990 50  0001 C CNN
+F 4 "C72041" H 6700 4990 50  0001 C CNN "LCSC"
 	1    6700 4990
 	1    0    0    1
@@
 F 2 "Resistor_SMD:R_0603_1608Metric" V 6930 4990 50  0001 C CNN
 F 3 "~" H 7000 4990 50  0001 C CNN
+F 4 "C4190" H 7000 4990 50  0001 C CNN "LCSC"
 	1    7000 4990
 	0    1    1    0
@@
 F 2 "Resistor_SMD:R_0603_1608Metric" V 6940 5180 50  0001 C CNN
 F 3 "~" H 7010 5180 50  0001 C CNN
+F 4 "C4190" H 7010 5180 50  0001 C CNN "LCSC"
 	1    7010 5180
 	0    1    1    0
@@
 F 2 "Resistor_SMD:R_0603_1608Metric" V 7250 2950 50  0001 C CNN
 F 3 "~" H 7320 2950 50  0001 C CNN
+F 4 "C25804" H 7320 2950 50  0001 C CNN "LCSC"
 	1    7320 2950
 	0    1    1    0
@@
 F 2 "LED_SMD:LED_0603_1608Metric" H 7020 2950 50  0001 C CNN
 F 3 "~" H 7020 2950 50  0001 C CNN
+F 4 "C72043" H 7020 2950 50  0001 C CNN "LCSC"
 	1    7020 2950
 	-1   0    0    1
@@
 F 2 "Capacitor_SMD:C_0603_1608Metric" H 5658 6880 50  0001 C CNN
 F 3 "~" H 5620 7030 50  0001 C CNN
+F 4 "C15849" H 5620 7030 50  0001 C CNN "LCSC"
 	1    5620 7030
 	-1   0    0    1
@@
 F 2 "Capacitor_SMD:C_0603_1608Metric" H 6588 6880 50  0001 C CNN
 F 3 "~" H 6550 7030 50  0001 C CNN
+F 4 "C15849" H 6550 7030 50  0001 C CNN "LCSC"
 	1    6550 7030
 	-1   0    0    1
@@
 F 2 "Resistor_SMD:R_0603_1608Metric" V 10400 2180 50  0001 C CNN
 F 3 "~" H 10470 2180 50  0001 C CNN
+F 4 "C25803" H 10470 2180 50  0001 C CNN "LCSC"
 	1    10470 2180
 	1    0    0    1
@@
 F 2 "Capacitor_SMD:C_1206_3216Metric" H 9528 2280 50  0001 C CNN
 F 3 "~" H 9490 2430 50  0001 C CNN
+F 4 "C59461" H 9490 2430 50  0001 C CNN "LCSC"
 	1    9490 2430
 	-1   0    0    1
@@
 F 2 "Capacitor_SMD:C_0603_1608Metric" H 10808 2030 50  0001 C CNN
 F 3 "~" H 10770 2180 50  0001 C CNN
+F 4 "C1653" H 10770 2180 50  0001 C CNN "LCSC"
 	1    10770 2180
 	-1   0    0    -1
@@
 F 2 "Capacitor_SMD:C_0603_1608Metric" H 10808 1730 50  0001 C CNN
 F 3 "~" H 10770 1880 50  0001 C CNN
+F 4 "C59461" H 10770 1880 50  0001 C CNN "LCSC"
 	1    10770 1880
 	-1   0    0    -1
@@
 F 2 "Capacitor_SMD:C_0603_1608Metric" H 10508 1730 50  0001 C CNN
 F 3 "~" H 10470 1880 50  0001 C CNN
+F 4 "C59461" H 10470 1880 50  0001 C CNN "LCSC"
 	1    10470 1880
 	-1   0    0    -1
@@
 F 2 "LED_SMD:LED_0603_1608Metric" H 9420 1560 50  0001 C CNN
 F 3 "~" H 9420 1560 50  0001 C CNN
+F 4 "C72038" H 9420 1560 50  0001 C CNN "LCSC"
 	1    9420 1560
 	1    0    0    -1
@@
 F 2 "Resistor_SMD:R_0603_1608Metric" V 9400 1010 50  0001 C CNN
 F 3 "~" H 9470 1010 50  0001 C CNN
+F 4 "C21190" H 9470 1010 50  0001 C CNN "LCSC"
 	1    9470 1010
 	-1   0    0    1
@@
 F 2 "Resistor_SMD:R_0603_1608Metric" V 9500 1880 50  0001 C CNN
 F 3 "~" H 9570 1880 50  0001 C CNN
+F 4 "C25804" H 9570 1880 50  0001 C CNN "LCSC"
 	1    9570 1880
 	-1   0    0    1
@@
 F 2 "Resistor_SMD:R_0603_1608Metric" V 7030 3450 50  0001 C CNN
 F 3 "~" H 7100 3450 50  0001 C CNN
+F 4 "C21189" H 7100 3450 50  0001 C CNN "LCSC"
 	1    7100 3450
 	0    1    1    0
@@
 F 2 "Resistor_SMD:R_0603_1608Metric" V 7030 3570 50  0001 C CNN
 F 3 "~" H 7100 3570 50  0001 C CNN
+F 4 "C21189" H 7100 3570 50  0001 C CNN "LCSC"
 	1    7100 3570
 	0    1    -1   0
@@
 F 2 "Resistor_SMD:R_0603_1608Metric" V 10550 2410 50  0001 C CNN
 F 3 "~" H 10620 2410 50  0001 C CNN
+F 4 "C31850" H 10620 2410 50  0001 C CNN "LCSC"
 	1    10620 2410
 	0    1    -1   0
@@
 F 2 "Resistor_SMD:R_0603_1608Metric" V 10700 2560 50  0001 C CNN
 F 3 "~" H 10770 2560 50  0001 C CNN
+F 4 "C21189" H 10770 2560 50  0001 C CNN "LCSC"
 	1    10770 2560
 	1    0    0    -1

Commit message: Detach Under Board
Parts:
- removed H5, H6, H7, H8: MountingHole, MountingHole:MountingHole_2.2mm_M2, symbol Mechanical:MountingHole
- removed U6, U7: ESP32FullConnector, KisonCommon:jtag1.27-10, symbol KisonCommon:ESP32FullConnector
Connections:
- net +3V3: now also C2.1, U5.50 (VREGIN)
Other:
- note added: "R24 to make it easier to modify VOut"
Changed lines of the file:
@@
 nRTS
-$Comp
-L KisonCommon:ESP32FullConnector U6
-U 1 1 605C8E21
-P 1420 6840
-F 0 "U6" H 1230 7264 50  0000 C CNN
-F 1 "ESP32FullConnector" H 1230 7173 50  0000 C CNN
-F 2 "KisonCommon:jtag1.27-10" H 1420 6840 50  0001 C CNN
-F 3 "" H 1420 6840 50  0001 C CNN
-	1    1420 6840
-	1    0    0    -1
-$EndComp
-$Comp
-L KisonCommon:ESP32FullConnector U7
-U 1 1 605CA8D0
-P 1430 7510
-F 0 "U7" H 1240 7934 50  0000 C CNN
-F 1 "ESP32FullConnector" H 1240 7843 50  0000 C CNN
-F 2 "KisonCommon:jtag1.27-10" H 1430 7510 50  0001 C CNN
-F 3 "" H 1430 7510 50  0001 C CNN
-	1    1430 7510
-	1    0    0    -1
-$EndComp
 $Comp
 L Mechanical:MountingHole H1
@@
 F 3 "" H 3320 5660 50  0001 C CNN
 	1    3320 5660
-	1    0    0    -1
-$EndComp
-$Comp
-L Mechanical:MountingHole H5
-U 1 1 605C59FE
-P 2500 6590
-F 0 "H5" H 2600 6636 50  0000 L CNN
-F 1 "MountingHole" H 2600 6545 50  0000 L CNN
-F 2 "MountingHole:MountingHole_2.2mm_M2" H 2500 6590 50  0001 C CNN
-F 3 "~" H 2500 6590 50  0001 C CNN
-	1    2500 6590
-	1    0    0    -1
-$EndComp
-$Comp
-L Mechanical:MountingHole H6
-U 1 1 605C5EED
-P 2520 6800
-F 0 "H6" H 2620 6846 50  0000 L CNN
-F 1 "MountingHole" H 2620 6755 50  0000 L CNN
-F 2 "MountingHole:MountingHole_2.2mm_M2" H 2520 6800 50  0001 C CNN
-F 3 "~" H 2520 6800 50  0001 C CNN
-	1    2520 6800
-	1    0    0    -1
-$EndComp
-$Comp
-L Mechanical:MountingHole H7
-U 1 1 605C6332
-P 2530 6990
-F 0 "H7" H 2630 7036 50  0000 L CNN
-F 1 "MountingHole" H 2630 6945 50  0000 L CNN
-F 2 "MountingHole:MountingHole_2.2mm_M2" H 2530 6990 50  0001 C CNN
-F 3 "~" H 2530 6990 50  0001 C CNN
-	1    2530 6990
-	1    0    0    -1
-$EndComp
-$Comp
-L Mechanical:MountingHole H8
-U 1 1 605C6637
-P 2540 7210
-F 0 "H8" H 2640 7256 50  0000 L CNN
-F 1 "MountingHole" H 2640 7165 50  0000 L CNN
-F 2 "MountingHole:MountingHole_2.2mm_M2" H 2540 7210 50  0001 C CNN
-F 3 "~" H 2540 7210 50  0001 C CNN
-	1    2540 7210
 	1    0    0    -1
 $EndComp
@@
 	1    0    0    -1
 $EndComp
+$Comp
+L power:+3V3 #PWR0153
+U 1 1 60865825
+P 3250 2080
+F 0 "#PWR0153" H 3250 1930 50  0001 C CNN
+F 1 "+3V3" V 3265 2208 50  0000 L CNN
+F 2 "" H 3250 2080 50  0001 C CNN
+F 3 "" H 3250 2080 50  0001 C CNN
+	1    3250 2080
+	1    0    0    -1
+$EndComp
+Connection ~ 3250 2080
+Text Notes 9210 2850 0    50   ~ 0
+R24 to make it easier to modify VOut
 $EndSCHEMATC

Commit message: V3
Parts:
- removed R22, R23: 0, Resistor_SMD:R_0603_1608Metric, symbol Device:R
- U1, U2: symbol KisonCommon:ESP32FullConnector -> KisonCommon:ESP32FullConnectorTX
Connections:
- net ESPRX is gone; now on net 2232TX: U1.10 (TX), U10.3 (IO2), U10.4 (IO2), U2.10 (TX)
- net ESPTX is gone; now on net 2232RX: U1.9 (RX), U10.1 (IO1), U10.6 (IO1), U2.9 (RX)
- net 3v3OUT: now also U1.1 (3V3), U2.1 (3V3); no longer U1.7 (3V3), U2.7 (3V3)
- net IO0: now also U13.3 (IO2), U13.4 (IO2); no longer U13.1 (IO1), U13.6 (IO1)
- net TCK: now also U1.3 (TCLK), U12.3 (IO2), U12.4 (IO2), U2.3 (TCLK); no longer U1.4 (TCLK), U12.1 (IO1), U12.6 (IO1), U2.4 (TCLK)
- net TDI: now also U1.5 (TDI), U2.5 (TDI); no longer U1.3 (TDI), U2.3 (TDI)
- net TDO: now also U1.4 (TDO), U11.1 (IO1), U11.6 (IO1), U2.4 (TDO); no longer U1.6 (TDO), U13.3 (IO2), U13.4 (IO2), U2.6 (TDO)
- net TMS: now also U1.6 (TMS), U12.1 (IO1), U12.6 (IO1), U2.6 (TMS); no longer U1.5 (TMS), U12.3 (IO2), U12.4 (IO2), U2.5 (TMS)
- net nTRST: now also U1.7 (nRST), U13.1 (IO1), U13.6 (IO1), U2.7 (nRST); no longer U1.1 (TRST), U11.1 (IO1), U11.6 (IO1), U2.1 (TRST)
Changed lines of the file:
@@
 $EndDescr
 $Comp
-L KisonCommon:ESP32FullConnector U1
+L KisonCommon:ESP32FullConnectorTX U1
 U 1 1 606238BC
 P 1200 1010
@@
 Text GLabel 6020 620  2    50   Input ~ 0
 nTRST
-Text GLabel 1220 800  2    50   Input ~ 0
+Text GLabel 1220 1070 2    50   Input ~ 0
 nTRST
-Text GLabel 1220 1450 2    50   Input ~ 0
+Text GLabel 1220 1720 2    50   Input ~ 0
 nTRST
 Text GLabel 800  1720 0    50   Input ~ 0
@@
 Text GLabel 800  1070 0    50   Input ~ 0
 IO0
+Text GLabel 1220 890  2    50   Input ~ 0
+TCK
+Text GLabel 1220 1540 2    50   Input ~ 0
+TCK
 Text GLabel 800  890  0    50   Input ~ 0
-TCK
+TDO
 Text GLabel 800  1540 0    50   Input ~ 0
-TCK
-Text GLabel 800  980  0    50   Input ~ 0
-TDO
-Text GLabel 800  1630 0    50   Input ~ 0
 TDO
 $Comp
@@
 	0    1    1    0
 $EndComp
-Text GLabel 1220 890  2    50   Input ~ 0
+Text GLabel 1220 980  2    50   Input ~ 0
 TDI
-Text GLabel 1220 1540 2    50   Input ~ 0
+Text GLabel 1220 1630 2    50   Input ~ 0
 TDI
-Text GLabel 1220 980  2    50   Input ~ 0
+Text GLabel 800  980  0    50   Input ~ 0
 TMS
-Text GLabel 1220 1630 2    50   Input ~ 0
+Text GLabel 800  1630 0    50   Input ~ 0
 TMS
 Text GLabel 6100 4280 2    50   Input ~ 0
@@
 	0    -1   -1   0
 $EndComp
-Text GLabel 1220 1070 2    50   Input ~ 0
+Text GLabel 1220 800  2    50   Input ~ 0
 3v3OUT
 $Comp
@@
 Wire Wire Line
 	10300 2330 10470 2330
-Text GLabel 1220 1720 2    50   Input ~ 0
+Text GLabel 1220 1450 2    50   Input ~ 0
 3v3OUT
 Text GLabel 8980 3130 1    50   Input ~ 0
@@
 	1    0    0    -1
 $EndComp
-Text GLabel 7980 3130 1    50   Input ~ 0
+Text GLabel 9390 4990 1    50   Input ~ 0
 nTRST
 $Comp
@@
 	1    0    0    -1
 $EndComp
-Text GLabel 7980 3330 3    50   Input ~ 0
+Text GLabel 9390 5190 3    50   Input ~ 0
 nTRST
 Text GLabel 8980 3330 3    50   Input ~ 0
@@
 	1    0    0    -1
 $EndComp
+Text GLabel 9390 3510 1    50   Input ~ 0
+TMS
 Text GLabel 10390 3510 1    50   Input ~ 0
-TMS
-Text GLabel 9390 3510 1    50   Input ~ 0
 TCK
-Text GLabel 9390 4990 1    50   Input ~ 0
+Text GLabel 10390 4990 1    50   Input ~ 0
 IO0
 $Comp
@@
 $EndComp
 $Comp
-L KisonCommon:USBLC6-2SC6-Power_Protection U10
-U 1 1 607A2348
-P 8450 4670
-F 0 "U10" H 8450 5351 50  0000 C CNN
-F 1 "USBLC6-2SC6-Power_Protection" H 8450 5280 50  0000 C CNN
-F 2 "KisonCommon:USBLC6-2P6-SOT666" H 7700 5070 50  0001 C CNN
-F 3 "" H 8650 5020 50  0001 C CNN
-	1    8450 4670
-	1    0    0    -1
-$EndComp
-$Comp
 L power:GND #PWR017
 U 1 1 607A4C4F
@@
 	1    0    0    -1
 $EndComp
+Text GLabel 9390 3710 3    50   Input ~ 0
+TMS
 Text GLabel 10390 3710 3    50   Input ~ 0
-TMS
-Text GLabel 9390 3710 3    50   Input ~ 0
 TCK
+Text GLabel 7980 3330 3    50   Input ~ 0
+TDO
+Text GLabel 7980 3130 1    50   Input ~ 0
+TDO
 Text GLabel 10390 5190 3    50   Input ~ 0
-TDO
-Text GLabel 10390 4990 1    50   Input ~ 0
-TDO
-Text GLabel 9390 5190 3    50   Input ~ 0
 IO0
 $Comp
@@
 Text GLabel 6100 3880 2    50   Input ~ 0
 2232TX
-Text GLabel 6950 3450 0    50   Input ~ 0
+Text GLabel 800  1810 0    50   Input ~ 0
 2232TX
-$Comp
-L Device:R R22
-U 1 1 607147ED
-P 7100 3450
-F 0 "R22" V 7100 3450 50  0000 C CNN
-F 1 "0" V 6984 3450 50  0000 C CNN
-F 2 "Resistor_SMD:R_0603_1608Metric" V 7030 3450 50  0001 C CNN
-F 3 "~" H 7100 3450 50  0001 C CNN
-F 4 "C21189" H 7100 3450 50  0001 C CNN "LCSC"
-	1    7100 3450
-	0    1    1    0
-$EndComp
-Text GLabel 7250 3450 2    50   Input ~ 0
-ESPRX
-$Comp
-L Device:R R23
-U 1 1 6071BB77
-P 7100 3570
-F 0 "R23" V 7100 3570 50  0000 C CNN
-F 1 "0" V 6984 3570 50  0000 C CNN
-F 2 "Resistor_SMD:R_0603_1608Metric" V 7030 3570 50  0001 C CNN
-F 3 "~" H 7100 3570 50  0001 C CNN
-F 4 "C21189" H 7100 3570 50  0001 C CNN "LCSC"
-	1    7100 3570
-	0    1    -1   0
-$EndComp
 Text GLabel 6100 3980 2    50   Input ~ 0
 2232RX
-Text GLabel 6950 3570 0    50   Input ~ 0
+Text GLabel 1220 1810 2    50   Input ~ 0
 2232RX
-Text GLabel 7250 3570 2    50   Input ~ 0
-ESPTX
-Text GLabel 1220 1160 2    50   Input ~ 0
-ESPTX
-Text GLabel 800  1160 0    50   Input ~ 0
-ESPRX
-Text GLabel 800  1810 0    50   Input ~ 0
-ESPRX
-Text GLabel 1220 1810 2    50   Input ~ 0
-ESPTX
 $Comp
 L power:+3V3 #PWR0152
@@
 	1    0    0    -1
 $EndComp
-Text GLabel 8950 4570 1    50   Input ~ 0
-ESPRX
-Text GLabel 7950 4570 1    50   Input ~ 0
-ESPTX
-Text GLabel 7950 4770 3    50   Input ~ 0
-ESPTX
-Text GLabel 8950 4770 3    50   Input ~ 0
-ESPRX
 Connection ~ 5400 1780
 Connection ~ 5300 1780
@@
 $EndComp
 $Comp
-L KisonCommon:ESP32FullConnector U2
+L KisonCommon:ESP32FullConnectorTX U2
 U 1 1 60623F40
 P 1200 1660
@@
 Text Notes 9210 2850 0    50   ~ 0
 R24 to make it easier to modify VOut
+Text GLabel 800  1160 0    50   Input ~ 0
+2232TX
+Text GLabel 1220 1160 2    50   Input ~ 0
+2232RX
+$Comp
+L KisonCommon:USBLC6-2SC6-Power_Protection U10
+U 1 1 607A2348
+P 8450 4670
+F 0 "U10" H 8450 5351 50  0000 C CNN
+F 1 "USBLC6-2SC6-Power_Protection" H 8450 5280 50  0000 C CNN
+F 2 "KisonCommon:USBLC6-2P6-SOT666" H 7700 5070 50  0001 C CNN
+F 3 "" H 8650 5020 50  0001 C CNN
+	1    8450 4670
+	1    0    0    -1
+$EndComp
+Text GLabel 7950 4770 3    50   Input ~ 0
+2232RX
+Text GLabel 8950 4770 3    50   Input ~ 0
+2232TX
+Text GLabel 8950 4570 1    50   Input ~ 0
+2232TX
+Text GLabel 7950 4570 1    50   Input ~ 0
+2232RX
 $EndSCHEMATC

Commit message: Based on esp-prog
Parts:
- added C16, C23: 1nf, Capacitor_SMD:C_0603_1608Metric, symbol Device:C
- added C24: 0.1uf/25v(10%), Capacitor_SMD:C_0603_1608Metric, symbol Device:C
- added C25, C26: 1uf/25v, Capacitor_SMD:C_0603_1608Metric, symbol Device:C
- added D1, D6: D_Schottky, Diode_SMD:D_SOD-523, symbol Device:D_Schottky
- added Q3: WST03P06, Package_TO_SOT_SMD:SOT-23, symbol Transistor_FET:SUD08P06-155L
- added R22, R23, R26, R27: 10k, Resistor_SMD:R_0603_1608Metric, symbol Device:R
- added R25: 0, Resistor_SMD:R_0603_1608Metric, symbol Device:R
- added SW2, SW3: SW_Push, KisonCommon:BTN-TS342A4P-WZ-C557592, symbol Switch:SW_Push
- added U6: SN74AHC125RGY, KisonCommon:VQFN-14_3.6x3.6x05P, symbol KisonCommon:SN74AHC125RGY
- added U7: 74AHC1GU04, Package_TO_SOT_SMD:SOT-353_SC-70-5, symbol 74xGxx:74AHC1GU04
- C17, C21: value 1uf -> 1uf/25v
Connections:
- net +3V3: now also C26.2, Q3.3 (S), R22.1, R23.1
- net GND: now also C16.2, C23.2, C24.1, C25.2, D6.2 (A), R27.1, SW2.1, SW3.1, U6.15 (TPAD), U6.7 (GND), U7.3 (GND)
- net IO0: no longer Q2.3 (C), U1.8 (IO0), U2.8 (IO0)
- net TCK: no longer U1.3 (TCLK), U2.3 (TCLK), U5.16 (ADBUS0)
- net TDI: no longer U1.5 (TDI), U2.5 (TDI), U5.17 (ADBUS1)
- net TDO: no longer U1.4 (TDO), U2.4 (TDO), U5.18 (ADBUS2)
- net TMS: no longer U1.6 (TMS), U2.6 (TMS), U5.19 (ADBUS3)
- net nTRST: no longer Q1.3 (C), U5.22 (ADBUS5)
- new net: D1.2 (A), R26.2, U7.4
- new net: C26.1, D6.1 (K), Q3.1 (G), R27.2
- new net ESP_EN: C23.1, Q1.3 (C), R23.2, SW3.2, U7.2
- new net ESP_EN_N: C25.1, D1.1 (K), R26.1, U6.1 (1~OE), U6.10 (3~OE), U6.13 (4~OE), U6.4 (2~OE)
- new net ESP_IO0: R25.2, U1.8 (IO0), U2.8 (IO0)
- new net ESP_IO0_B: C16.1, Q2.3 (C), R22.2, R25.1, SW2.2
- new net ESP_TCK: U1.3 (TCLK), U2.3 (TCLK), U6.11 (4Y)
- new net ESP_TDI: U1.5 (TDI), U2.5 (TDI), U6.8 (3Y)
- new net ESP_TDO: U1.4 (TDO), U2.4 (TDO), U6.5 (2A)
- new net ESP_TMS: U1.6 (TMS), U2.6 (TMS), U6.3 (1Y)
- new net FT_TCK: U5.16 (ADBUS0), U6.12 (4A)
- new net FT_TDI: U5.17 (ADBUS1), U6.9 (3A)
- new net FT_TDO: U5.18 (ADBUS2), U6.6 (2Y)
- new net FT_TMS: U5.19 (ADBUS3), U6.2 (1A)
- new net VCC: C24.2, Q3.2 (D), U6.14 (VCC), U7.5 (VCC)
Other:
- moved on the sheet: C1, C10, C11, C12, C13, C14, C15, C17, C18, C19, C2, C20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
