File: ft2232h_esp32.sch (KiCad schematic (older format))
At the start: 70 parts, among them J1 USB_C_Receptacle_USB2.0, Q1 S8050, Q2 S8050, SW1 SW_SPDT, U1 ESP32FullConnector, U10 USBLC6-2SC6-Power_Protection, U11 USBLC6-2SC6-Power_Protection, U12 USBLC6-2SC6-Power_Protection, U13 USBLC6-2SC6-Power_Protection, U2 ESP32FullConnector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

Commit message: V4
Fix BJT bug
Parts:
- Q1, Q2: value S8050 -> SS8050; symbol Transistor_BJT:S8050 -> Transistor_BJT:2N3055
Connections:
- net nDTR: now also Q2.2 (E); no longer Q2.1 (E)
- net nRTS: now also Q1.2 (E); no longer Q1.1 (E)
- net at R13.1: now also Q1.1 (B); no longer Q1.2 (B)
- net at R14.1: now also Q2.1 (B); no longer Q2.2 (B)
Changed lines of the file:
@@
 nTRST
 $Comp
-L Transistor_BJT:S8050 Q1
+L Transistor_BJT:2N3055 Q1
 U 1 1 60683C3F
 P 5920 820
 F 0 "Q1" H 6110 866 50  0000 L CNN
-F 1 "S8050" H 6110 775 50  0000 L CNN
+F 1 "SS8050" H 6110 775 50  0000 L CNN
 F 2 "Package_TO_SOT_SMD:SOT-23" H 6120 745 50  0001 L CIN
 F 3 "http://www.unisonic.com.tw/datasheet/S8050.pdf" H 5920 820 50  0001 L CNN
@@
 $EndComp
 $Comp
-L Transistor_BJT:S8050 Q2
+L Transistor_BJT:2N3055 Q2
 U 1 1 60684A60
 P 5920 1340
 F 0 "Q2" H 6110 1294 50  0000 L CNN
-F 1 "S8050" H 6110 1385 50  0000 L CNN
+F 1 "SS8050" H 6110 1385 50  0000 L CNN
 F 2 "Package_TO_SOT_SMD:SOT-23" H 6120 1265 50  0001 L CIN
 F 3 "http://www.unisonic.com.tw/datasheet/S8050.pdf" H 5920 1340 50  0001 L CNN
